File: sedsna-kicad/sedsna.kicad_sch (KiCad schematic)
At the start: 47 parts, among them J1 Conn_01x03, J10 Conn_01x03, J2 Conn_01x03, J3 Servos_Rudder/Elevator, J4 L_Aileron, J5 USB4105-GF-A, J6 R_Aileron, J7 Prop, J8 Antenna, J9 Conn_01x03, U2 ESP32-C3, U4 Magnetometer, U5 IMU, U6 LDL1117S33R

Commit message: Signal pins from receiver
Connections:
- net +3.3V: now also J1.2 (Pin_2), J10.2 (Pin_2), J2.2 (Pin_2), J9.2 (Pin_2); no longer J1.1 (Pin_1), J10.1 (Pin_1), J2.1 (Pin_1), J9.1 (Pin_1)
- net Earth: now also J1.1 (Pin_1), J10.1 (Pin_1), J2.1 (Pin_1), J9.1 (Pin_1)
- net Channel_4: now reaches J10.3 (Pin_3)
- net Channel_4: now also U2.16 (GPIO10)
- net Channel_2: now reaches J2.3 (Pin_3)
- net Channel_2: now also U2.5 (XTAL_32K_N)
- net Channel_3: now reaches U2.15 (GPIO9)
- net Channel_3: now also J9.3 (Pin_3)
- net Channel_1: now reaches U2.4 (XTAL_32K_P)
- net Channel_1: now also J1.3 (Pin_3)
- no-connect marks 17 -> 15

Commit message: schematic done?
all pcb import errors cleared at least
Parts:
- removed BAT1: Screw_Terminal_01x02, TerminalBlock:TerminalBlock_bornier-2_P5.08mm, symbol TR3_V1:Screw_Terminal_01x02
- added BAT1: Conn_01x02, sedsna:CONN_SDA_42002-xxxxx_02_MOL, symbol Connector_Generic:Conn_01x02
- J1, J10, J2, J9: footprint (none) -> Connector_PinHeader_2.54mm:PinHeader_1x03_P2.54mm_Vertical
- U2: footprint Connector_Coaxial:SMA_Molex_73251-1153_EdgeMount_Horizontal -> sedsna:QFN32_5X5_EXP
Connections:
- net at BR1.2: now also BAT1.1 (Pin_1)
- net at BR1.3: now also BAT1.2 (Pin_2)
Other:
- moved on the sheet: C8, C9, J1, J10, J2, J3, J4, J6, J7, J8, J9, L1

Commit message: pcb layout started
Parts:
- removed BAT1: Conn_01x02, sedsna:CONN_SDA_42002-xxxxx_02_MOL, symbol Connector_Generic:Conn_01x02
- removed BR1: Z4DGP406L-HF, TR3_V1:Z4DGP406L-HF_footprint_N, symbol TR3_V1:Z4DGP406L-HF
- removed J8: Antenna, sedsna:CONN_142-0701-801, symbol Connector:Conn_Coaxial_Small
- added AE1: Antenna, TR3_V1:GRADCONN_RFPC-SMA28-F, symbol TR3_V1:RFPC-SMA28-F
- added J11: BAT1, sedsna:SHDR3W166P0X635_1X3_2032X762X1397P, symbol Connector_Generic:Conn_01x03
- J4, J6, J7: footprint sedsna:CONN_SDA_42002-xxxxx_03_MOL -> sedsna:SHDR3W166P0X635_1X3_2032X762X1397P
Connections:
- net +7.4V: now also J11.1 (Pin_1), J11.3 (Pin_3)
- net Earth: now also AE1.G1, AE1.G2, AE1.G3, AE1.G4, J11.2 (Pin_2)
- net at C8.1, L1.2: now also AE1.1
Other:
- moved on the sheet: C1, C15, C19, C2, C6, ENABLE2, J5, PWR1, R16, R17, R18, R19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

Commit message: mounting holes added
Parts:
- added H1, H2, H3, H4: MountingHole, sedsna:mounting_hole, symbol Mechanical:MountingHole
Other:
- note added: "Mounting Holes"

Commit message: Finished layout
Parts:
- removed ENABLE2: Enable Switch, TR3_V1:SW_DS04-254-2-01BK-SMT, symbol TR3_V1:SW_DIP_x01
- removed J1, J10, J2, J9: Conn_01x03, Connector_PinHeader_2.54mm:PinHeader_1x03_P2.54mm_Vertical, symbol Connector_Generic:Conn_01x03
- added J1: (no value), sedsna:Conn_04x03, symbol JM-Lib:Conn_03x04
- C7: footprint Capacitor_SMD:C_01005_0402Metric_Pad0.57x0.30mm_HandSolder -> TR3_V1:CAP_CL05_SAM
Connections:
- net USB_D+ is gone; now on net Earth: J5.A6 (DP1), J5.B6 (DP2), U2.26 (GPIO19)
- net +3.3V: now also R7.1, J1.11, J1.2, J1.5, J1.8
- net Channel_1: now also J1.3
- net Channel_2: now also J1.6
- net Channel_3: now also J1.9
- net Channel_4: now also J1.12
- net Earth: now also U2.27 (U0RXD), J1.1, J1.10, J1.4, J1.7
- net +7.4V renamed +6.6V
- net +6.6V: no longer J11.3 (Pin_3)
