File: kicad/sedsna-kicad/sedsna.kicad_pcb (KiCad board)
At the start: 4 copper layers, 40 x 91 mm, 46 parts, among them J11 BAT1, J3 Servos_Rudder/Elevator, J4 L_Aileron, J5 USB4105-GF-A, J6 R_Aileron, J7 Prop, U2 ESP32-C3, U4 Magnetometer, U5 IMU, U6 LDL1117S33R

Commit message: did some routing
Parts:
- moved R2 1.41 mm to (126.2, 67.7)
- moved C2 1.41 mm to (122.6, 71.2)
- moved XTAL1 1.41 mm to (123.9, 69.8)
- moved C1 1.41 mm to (125.2, 68.5)
- moved U6 1.15 mm to (118.8, 74.8)
- moved C6 0.17 mm to (119.8, 71.5)
- renumbered PWR to PWR1, RESET to RESET1, STAT to STAT1
Connections:
- J1 pad 11: +3.3V -> +6.6V
- J1 pad 2: +3.3V -> +6.6V
- J1 pad 5: +3.3V -> +6.6V
- J1 pad 8: +3.3V -> +6.6V
- J5 pad A6: Earth -> /USB_D+
- J5 pad B6: Earth -> /USB_D+
- U2 pad 26: Earth -> /USB_D+
Routing:
- net Earth: track 0.00 -> 93.1 mm, vias 0 -> 6
- net +6.6V: track 0.00 -> 84.7 mm, vias 0 -> 1
- net +3.3V: track 0.00 -> 45.7 mm, vias 0 -> 7
- net /USB_D-: track 0.00 -> 35.1 mm, vias 0 -> 2
- net /USB_D+: track 0.00 -> 30.0 mm, vias 0 -> 2
- net /VBUS: track 0.00 -> 15.5 mm, vias 0 -> 1
- net Net-(STAT1-A): track 0.00 -> 14.5 mm
- net /I2C_SCL: track 0.00 -> 8.79 mm, vias 0 -> 2
- net /I2C_SDA: track 0.00 -> 6.76 mm
- net Net-(U2-CHIP_EN): track 0.00 -> 5.57 mm
- net Net-(U2-XTAL_N): track 0.00 -> 4.97 mm
- net Net-(U2-XTAL_P): track 0.00 -> 3.64 mm
- net Net-(STAT1-K): track 0.00 -> 2.88 mm, vias 0 -> 1
- net Net-(B1-SDO): track 0.00 -> 2.78 mm, vias 0 -> 1
- net Net-(XTAL1-IN/OUT): track 0.00 -> 2.71 mm
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
Commit message: PCB draft, Lily needs to do antenna stuff
Parts:
- moved AE1 1.98 mm to (132.2, 62.4)
- moved C8 1.49 mm to (127.2, 61.8)
- moved L1 1.44 mm to (126.3, 63.1)
- moved C9 1.42 mm to (125.5, 64.5)
Connections:
- U2 pad 15: /Channel_3 -> /Channel_2
- U2 pad 16: /Channel_4 -> /Channel_1
- U2 pad 4: /Channel_1 -> /Channel_4
- U2 pad 5: /Channel_2 -> /Channel_3
Routing:
- net /CTR_Rudder: track 0.00 -> 74.3 mm, vias 0 -> 2
- net /CTR_L_Ail: track 0.00 -> 69.0 mm, vias 0 -> 2
- net /CTR_Elevator: track 0.00 -> 66.2 mm, vias 0 -> 3
- net /CTR_Prop: track 0.00 -> 63.5 mm, vias 0 -> 2
- net +6.6V: track 84.7 -> 144.4 mm
- net /CTR_R_Ail: track 0.00 -> 58.8 mm, vias 0 -> 2
- net Net-(U2-CHIP_EN): track 5.57 -> 61.2 mm, vias 0 -> 2
- net /I2C_SCL: track 8.79 -> 45.9 mm, vias 2 -> 6
- net /I2C_SDA: track 6.76 -> 32.9 mm, vias 0 -> 3
- net /Channel_1: track 0.00 -> 24.4 mm
- net /Channel_3: track 0.00 -> 22.7 mm
- net /Channel_2: track 0.00 -> 21.6 mm
- net /Channel_4: track 0.00 -> 21.0 mm
- net +3.3V: track 45.7 -> 59.6 mm, vias 7 -> 14
- net Net-(AE1-Pad1): track 3.77 -> 0.00 mm
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