File: kicad/sedsna-kicad/sedsna.kicad_pcb (KiCad board)
At the start: 4 copper layers, 40 x 91 mm, 46 parts, among them J11 BAT1, J3 Servos_Rudder/Elevator, J4 L_Aileron, J5 USB4105-GF-A, J6 R_Aileron, J7 Prop, U2 ESP32-C3, U4 Magnetometer, U5 IMU, U6 LDL1117S33R

Commit message: worked on antenna trace
worked on antenna trace :)
Parts:
- moved AE1 1.94 mm to (131.9, 60.5)
- moved C8 1.42 mm to (126.0, 60.9)
- moved C9 1.42 mm to (124.5, 63.6)
- moved L1 1.42 mm to (125.2, 62.2)
Routing:
- net Earth: track 92.4 -> 77.4 mm, vias 55 -> 48
- net /I2C_SCL: track 45.9 -> 36.9 mm
- net +3.3V: track 59.6 -> 52.3 mm
- net /ANT: track 1.55 -> 2.75 mm
- net Net-(AE1-Pad1): track 0.00 -> 0.96 mm

Commit message: Finished ! (?) Pretty sure!
:)
Routing:
- net Earth: track 77.4 -> 98.3 mm, vias 48 -> 61
- net Net-(PWR1-K): track 0.00 -> 2.70 mm, vias 0 -> 1
Other:
- board text added: "my antennae are not for radio!!"
