File: kicad/sedsna-kicad/sedsna.kicad_sch (KiCad schematic)
At the start: 46 parts, among them J11 BAT1, J3 Servos_Rudder/Elevator, J4 L_Aileron, J5 USB4105-GF-A, J6 R_Aileron, J7 Prop, U2 ESP32-C3, U4 Magnetometer, U5 IMU, U6 LDL1117S33R

Commit message: did some routing
Connections:
- net +3.3V: no longer J1.11, J1.2, J1.5, J1.8
- net +6.6V: now also J1.11, J1.2, J1.5, J1.8
- net Earth: no longer J5.A6 (DP1), J5.B6 (DP2), U2.26 (GPIO19)
- new net USB_D+: J5.A6 (DP1), J5.B6 (DP2), U2.26 (GPIO19)
Changed lines of the file:
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@@
 	)
 	(junction
-		(at 141.605 134.62)
-		(diameter 0)
-		(color 0 0 0 0)
-	)
-	(junction
 		(at 323.85 85.09)
 		(diameter 0)
@@
 	(wire
 		(pts
-			(xy 141.605 134.62) (xy 141.605 140.335)
+			(xy 141.605 132.08) (xy 141.605 140.335)
 		)
 		(stroke
@@
 	(wire
 		(pts
-			(xy 141.605 132.08) (xy 141.605 134.62)
-		)
-		(stroke
-			(width 0)
-			(type default)
-		)
-	)
-	(wire
-		(pts
 			(xy 36.83 106.68) (xy 36.83 124.46)
 		)
@@
 	(wire
 		(pts
-			(xy 129.54 134.62) (xy 141.605 134.62)
-		)
-		(stroke
-			(width 0)
-			(type default)
-		)
-	)
-	(wire
-		(pts
 			(xy 55.88 66.04) (xy 57.15 66.04)
 		)
@@
 	(wire
 		(pts
+			(xy 129.54 134.62) (xy 138.43 134.62)
+		)
+		(stroke
+			(width 0)
+			(type default)
+		)
+	)
+	(wire
+		(pts
 			(xy 332.105 127) (xy 335.915 127)
 		)
@@
 			)
 		)
-		(property "Value" "+3.3V"
-			(at 351.155 137.1599 90)
+		(property "Value" "+6.6V"
+			(at 350.52 137.1599 90)
 			(show_name no)
 			(do_not_autoplace no)
@@
 			)
 		)
-		(property "Value" "+3.3V"
-			(at 351.155 126.9999 90)
+		(property "Value" "+6.6V"
+			(at 350.52 126.9999 90)
 			(show_name no)
 			(do_not_autoplace no)
@@
 		(in_pos_files yes)
 		(dnp no)
-		(fields_autoplaced yes)
 		(property "Reference" "#PWR018"
 			(at 335.915 137.16 0)
@@
 			)
 		)
-		(property "Value" "+3.3V"
-			(at 328.295 137.1599 90)
+		(property "Value" "+6.6V"
+			(at 327.152 136.906 90)
 			(show_name no)
 			(do_not_autoplace no)
@@
 					(size 1.27 1.27)
 				)
-				(justify left)
 			)
 		)
@@
 		(in_pos_files yes)
 		(dnp no)
-		(fields_autoplaced yes)
 		(property "Reference" "#PWR017"
 			(at 335.915 127 0)
@@
 			)
 		)
-		(property "Value" "+3.3V"
-			(at 328.295 126.9999 90)
+		(property "Value" "+6.6V"
+			(at 326.644 126.746 90)
 			(show_name no)
 			(do_not_autoplace no)
@@
 					(size 1.27 1.27)
 				)
-				(justify left)
 			)
 		)

Commit message: PCB draft, Lily needs to do antenna stuff
Connections:
- net Channel_1: now also U2.16 (GPIO10); no longer U2.4 (XTAL_32K_P)
- net Channel_2: now also U2.15 (GPIO9); no longer U2.5 (XTAL_32K_N)
- net Channel_3: now also U2.5 (XTAL_32K_N); no longer U2.15 (GPIO9)
- net Channel_4: now also U2.4 (XTAL_32K_P); no longer U2.16 (GPIO10)
Changed lines of the file:
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@@
 		)
 	)
-	(label "Channel_1"
+	(label "Channel_4"
 		(at 57.15 127 0)
 		(effects
@@
 		)
 	)
-	(label "Channel_3"
+	(label "Channel_2"
 		(at 57.15 153.67 0)
 		(effects
@@
 		)
 	)
-	(label "Channel_2"
+	(label "Channel_3"
 		(at 57.15 129.54 0)
 		(effects
@@
 		)
 	)
-	(label "Channel_4"
+	(label "Channel_1"
 		(at 57.15 156.21 0)
 		(effects
